File: pcb/esp32_blinds_controller.kicad_pcb (KiCad board)
At the start: 2 copper layers, 100 x 83.2 mm, 42 parts, among them J1 Conn_01x05_Pin, K1 G5LE-1, K2 G5LE-1, K3 G5LE-1, K4 G5LE-1, U1 MCP23008-xP, U2 ULN2003A, U3 R-78C3.3-1.0, U4 PC817, U5 PC817, U6 PC817, U7 PC817

Commit message: update
Connections:
- U1 pad 6: unconnected-(U1-~{RESET}-Pad6) -> +3V3
Routing:
- net +3V3: track 178.1 -> 189.1 mm
