File: pcb/esp32_blinds_controller.kicad_pcb (KiCad board)
At the start: 2 copper layers, 100 x 83.2 mm, 42 parts, among them J1 Conn_01x05_Pin, K1 G5LE-1, K2 G5LE-1, K3 G5LE-1, K4 G5LE-1, U1 MCP23008-xP, U2 ULN2003A, U3 R-78C3.3-1.0, U4 PC817, U5 PC817, U6 PC817, U7 PC817

Commit message: update
Parts:
- K1, K2, K3, K4: value G5LE-1 -> LEG-24
- MOD1: value ~ -> 4x TerminalBlock_Phoenix_MKDS-1,5-8_1x08_P5.00mm + ZD1006
- U3: value R-78C3.3-1.0 -> R-78E3.3-1.0
- U4, U5, U6, U7: value PC817 -> EL817
Connections:
- U2 pad 1: /DN1 -> unconnected-(U2-I1-Pad1)
- U2 pad 2: /UP1 -> unconnected-(U2-I2-Pad2)
- U2 pad 3: /DN2 -> unconnected-(U2-I3-Pad3)
- U2 pad 5: GND -> /DN2
- U2 pad 6: GND -> /UP1
- U2 pad 7: GND -> /DN1
Routing:
- net /DN1: track 21.7 -> 40.3 mm
- net /UP1: track 22.9 -> 33.2 mm
- net GND: track 7.62 -> 0.00 mm
- net /DN2: track 23.5 -> 29.4 mm, vias 0 -> 1
- net /UP2: track 22.6 -> 23.5 mm, vias 0 -> 1
Changed lines of the file:
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@@
 		)
 	)
-	(property "Revision" "V0.1")
+	(property "Revision" "V0.2")
 	(net 0 "")
 	(net 1 "Net-(K1-Pad4)")
@@
 	(net 42 "Net-(R11-Pad1)")
 	(net 43 "/IN3_H")
+	(net 44 "unconnected-(U2-I1-Pad1)")
+	(net 45 "unconnected-(U2-I3-Pad3)")
+	(net 46 "unconnected-(U2-I2-Pad2)")
 	(footprint "Capacitor_THT:CP_Radial_D8.0mm_P3.50mm"
 		(layer "F.Cu")
@@
 			)
 		)
-		(property "Value" "PC817"
+		(property "Value" "EL817"
 			(at 3.81 4.87 90)
 			(layer "F.Fab")
@@
 			)
 		)
-		(property "Datasheet" "http://www.soselectronic.cz/a_info/resource/d/pc817.pdf"
+		(property "Datasheet" "http://www.everlight.com/file/ProductFile/EL817.pdf"
 			(at 0 0 -90)
 			(unlocked yes)
@@
 			)
 		)
-		(property "Description" "DC Optocoupler, Vce 35V, CTR 50-300%, DIP-4"
+		(property "Description" "DC Optocoupler, Vce 35V, DIP-4"
 			(at 0 0 -90)
 			(unlocked yes)
@@
 			)
 		)
-		(property "Value" "G5LE-1"
+		(property "Value" "LEG-24"
 			(at 0 20.95 0)
 			(layer "F.Fab")
@@
 			(layers "*.Cu" "*.Mask")
 			(remove_unused_layers no)
-			(net 19 "/DN1")
+			(net 44 "unconnected-(U2-I1-Pad1)")
 			(pinfunction "I1")
-			(pintype "input")
+			(pintype "input+no_connect")
 		)
 		(pad "2" thru_hole oval
@@
 			(layers "*.Cu" "*.Mask")
 			(remove_unused_layers no)
-			(net 20 "/UP1")
+			(net 46 "unconnected-(U2-I2-Pad2)")
 			(pinfunction "I2")
-			(pintype "input")
+			(pintype "input+no_connect")
 		)
 		(pad "3" thru_hole oval
@@
 			(layers "*.Cu" "*.Mask")
 			(remove_unused_layers no)
-			(net 21 "/DN2")
+			(net 45 "unconnected-(U2-I3-Pad3)")
 			(pinfunction "I3")
-			(pintype "input")
+			(pintype "input+no_connect")
 		)
 		(pad "4" thru_hole oval
@@
 			(layers "*.Cu" "*.Mask")
 			(remove_unused_layers no)
-			(net 2 "GND")
+			(net 21 "/DN2")
 			(pinfunction "I5")
 			(pintype "input")
@@
 			(layers "*.Cu" "*.Mask")
 			(remove_unused_layers no)
-			(net 2 "GND")
+			(net 20 "/UP1")
 			(pinfunction "I6")
 			(pintype "input")
@@
 			(layers "*.Cu" "*.Mask")
 			(remove_unused_layers no)
-			(net 2 "GND")
+			(net 19 "/DN1")
 			(pinfunction "I7")
 			(pintype "input")
@@
 			(net 24 "unconnected-(U2-O3-Pad14)")
 			(pinfunction "O3")
-			(pintype "open_collector")
+			(pintype "open_collector+no_connect")
 		)
 		(pad "15" thru_hole oval
@@
 			(net 17 "unconnected-(U2-O2-Pad15)")
 			(pinfunction "O2")
-			(pintype "open_collector")
+			(pintype "open_collector+no_connect")
 		)
 		(pad "16" thru_hole oval
@@
 			(net 23 "unconnected-(U2-O1-Pad16)")
 			(pinfunction "O1")
-			(pintype "open_collector")
+			(pintype "open_collector+no_connect")
 		)
 		(model "${KICAD8_3DMODEL_DIR}/Package_DIP.3dshapes/DIP-16_W7.62mm.wrl"
@@
 			)
 		)
-		(property "Value" "G5LE-1"
+		(property "Value" "LEG-24"
 			(at 0 20.95 0)
 			(layer "F.Fab")
@@
 			)
 		)
-		(property "Value" "PC817"
+		(property "Value" "EL817"
 			(at 3.81 4.87 90)
 			(layer "F.Fab")
@@
 			)
 		)
-		(property "Datasheet" "http://www.soselectronic.cz/a_info/resource/d/pc817.pdf"
+		(property "Datasheet" "http://www.everlight.com/file/ProductFile/EL817.pdf"
 			(at 0 0 -90)
 			(unlocked yes)
@@
 			)
 		)
-		(property "Description" "DC Optocoupler, Vce 35V, CTR 50-300%, DIP-4"
+		(property "Description" "DC Optocoupler, Vce 35V, DIP-4"
 			(at 0 0 -90)
 			(unlocked yes)
@@
 			)
 		)
-		(property "Value" "G5LE-1"
+		(property "Value" "LEG-24"
 			(at 0 20.95 0)
 			(layer "F.Fab")
@@
 			)
 		)
-		(property "Value" "PC817"
+		(property "Value" "EL817"
 			(at 3.81 4.87 90)
 			(layer "F.Fab")
@@
 			)
 		)
-		(property "Datasheet" "http://www.soselectronic.cz/a_info/resource/d/pc817.pdf"
+		(property "Datasheet" "http://www.everlight.com/file/ProductFile/EL817.pdf"
 			(at 0 0 -90)
 			(unlocked yes)
@@
 			)
 		)
-		(property "Description" "DC Optocoupler, Vce 35V, CTR 50-300%, DIP-4"
+		(property "Description" "DC Optocoupler, Vce 35V, DIP-4"
 			(at 0 0 -90)
 			(unlocked yes)
@@
 			)
 		)
-		(property "Value" "~"
+		(property "Value" "4x TerminalBlock_Phoenix_MKDS-1,5-8_1x08_P5.00mm + ZD1006"
 			(at 3.875 0.98 0)
 			(unlocked yes)
@@
 			)
 		)
-		(property "Value" "PC817"
+		(property "Value" "EL817"
 			(at 3.81 4.87 90)
 			(layer "F.Fab")
@@
 			)
 		)
-		(property "Datasheet" "http://www.soselectronic.cz/a_info/resource/d/pc817.pdf"
+		(property "Datasheet" "http://www.everlight.com/file/ProductFile/EL817.pdf"
 			(at 0 0 -90)
 			(unlocked yes)
@@
 			)
 		)
-		(property "Description" "DC Optocoupler, Vce 35V, CTR 50-300%, DIP-4"
+		(property "Description" "DC Optocoupler, Vce 35V, DIP-4"
 			(at 0 0 -90)
 			(unlocked yes)
@@
 			)
 		)
-		(property "Value" "R-78C3.3-1.0"
+		(property "Value" "R-78E3.3-1.0"
 			(at 2.54 3 0)
 			(layer "F.Fab")
@@
 			)
 		)
-		(property "Datasheet" "https://www.recom-power.com/pdf/Innoline/R-78Cxx-1.0.pdf"
+		(property "Datasheet" "https://www.recom-power.com/pdf/Innoline/R-78Exx-1.0.pdf"
 			(at 0 0 0)
 			(unlocked yes)
@@
 			)
 		)
-		(property "Description" "1A Step-Down DC/DC-Regulator, 6-42V input, 3.3V fixed Output Voltage, LM78xx replacement, -40°C to +85°C, SIP3"
+		(property "Description" "1A Step-Down DC/DC-Regulator, 6-28V input, 3.3V fixed Output Voltage, LM78xx replacement, -40°C to +85°C, SIP3"
 			(at 0 0 0)
 			(unlocked yes)
@@
 			)
 		)
-		(property "Value" "G5LE-1"
+		(property "Value" "LEG-24"
 			(at 0 20.95 0)
 			(layer "F.Fab")
@@
 		(net 1)
 	)
-	(segment
-		(start 117.22 84.8)
-		(end 124.84 84.8)
-		(width 0.5)
-		(layer "F.Cu")
-		(net 2)
-	)
 	(via
 		(at 152.7 88.1)
@@
 	)
 	(segment
-		(start 152.98 92.42)
-		(end 152.98 91.48)
+		(start 119.76 84.8)
+		(end 119.76 82.94)
+		(width 0.5)
+		(layer "F.Cu")
+		(net 19)
+	)
+	(segment
+		(start 120.7 82)
+		(end 137.6 82)
 		(width 0.5)
 		(layer "F.Cu")
@@
 	(segment
 		(start 149.1 87.6)
-		(end 140.2 87.6)
+		(end 144.1 87.6)
 		(width 0.5)
 		(layer "F.Cu")
@@
 	)
 	(segment
-		(start 137.4 84.8)
-		(end 135 84.8)
+		(start 152.98 92.42)
+		(end 152.98 91.48)
 		(width 0.5)
 		(layer "F.Cu")
@@
 	)
 	(segment
-		(start 140.2 87.6)
-		(end 137.4 84.8)
+		(start 119.76 82.94)
+		(end 120.7 82)
 		(width 0.5)
 		(layer "F.Cu")
@@
 	)
 	(segment
-		(start 148.1 88.9)
-		(end 139.5 88.9)
+		(start 143.2 87.6)
+		(end 144.1 87.6)
 		(width 0.5)
 		(layer "F.Cu")
-		(net 20)
+		(net 19)
 	)
 	(segment
-		(start 139.5 88.9)
-		(end 137.8 87.2)
+		(start 137.6 82)
+		(end 143.2 87.6)
 		(width 0.5)
 		(layer "F.Cu")
-		(net 20)
+		(net 19)
 	)
 	(segment
@@
 	)
 	(segment
-		(start 137.8 87.2)
-		(end 133 87.2)
+		(start 150.44 92.42)
+		(end 150.44 91.24)
 		(width 0.5)
 		(layer "F.Cu")
@@
 	)
 	(segment
-		(start 132.46 86.66)
-		(end 132.46 84.8)
+		(start 148.1 88.9)
+		(end 142.4 88.9)
 		(width 0.5)
 		(layer "F.Cu")
@@
 	)
 	(segment
-		(start 150.44 92.42)
-		(end 150.44 91.24)
+		(start 141 87.5)
+		(end 123 87.5)
 		(width 0.5)
 		(layer "F.Cu")
@@
 	)
 	(segment
-		(start 133 87.2)
-		(end 132.46 86.66)
+		(start 123 87.5)
+		(end 122.3 86.8)
 		(width 0.5)
 		(layer "F.Cu")
@@
 	)
 	(segment
-		(start 138.9 90.1)
-		(end 137.3 88.5)
+		(start 122.3 86.8)
+		(end 122.3 84.8)
 		(width 0.5)
 		(layer "F.Cu")
-		(net 21)
+		(net 20)
 	)
 	(segment
-		(start 146.9 90.1)
-		(end 138.9 90.1)
+		(start 142.4 88.9)
+		(end 141 87.5)
 		(width 0.5)
 		(layer "F.Cu")
-		(net 21)
+		(net 20)
 	)
 	(segment
 		(start 147.9 91.1)
-		(end 146.9 90.1)
+		(end 147.9 92.42)
 		(width 0.5)
 		(layer "F.Cu")
@@
 	)
 	(segment
-		(start 129.92 87.52)
-		(end 129.92 84.8)
+		(start 146.9 90.1)
+		(end 147.9 91.1)
 		(width 0.5)
 		(layer "F.Cu")
@@
 	)
 	(segment
-		(start 147.9 92.42)
-		(end 147.9 91.1)
+		(start 141.7 90.1)
+		(end 146.9 90.1)
 		(width 0.5)
 		(layer "F.Cu")
@@
 	)
 	(segment
-		(start 130.9 88.5)
-		(end 129.92 87.52)
+		(start 140.5 88.9)
+		(end 141.7 90.1)
 		(width 0.5)
 		(layer "F.Cu")
@@
 	)
 	(segment
-		(start 137.3 88.5)
-		(end 130.9 88.5)
+		(start 124.84 88.9)
+		(end 140.5 88.9)
 		(width 0.5)
 		(layer "F.Cu")
 		(net 21)
 	)
+	(via
+		(at 124.84 88.9)
+		(size 0.65)
+		(drill 0.3)
+		(layers "F.Cu" "B.Cu")
+		(net 21)
+	)
 	(segment
-		(start 139.02 92.42)
-		(end 136.6 90)
+		(start 124.84 88.9)
+		(end 124.84 84.8)
+		(width 0.5)
+		(layer "B.Cu")
+		(net 21)
+	)
+	(segment
+		(start 142.02 92.42)
+		(end 145.36 92.42)
 		(width 0.5)
 		(layer "F.Cu")
@@
 	)
 	(segment
-		(start 127.38 87.38)
-		(end 127.38 84.8)
+		(start 139.6 90)
+		(end 142.02 92.42)
 		(width 0.5)
 		(layer "F.Cu")
@@
 	)
 	(segment
-		(start 136.6 90)
-		(end 130 90)
+		(start 128.5 90)
+		(end 139.6 90)
 		(width 0.5)
 		(layer "F.Cu")
 		(net 22)
 	)
+	(via
+		(at 128.5 90)
+		(size 0.65)
+		(drill 0.3)
+		(layers "F.Cu" "B.Cu")
+		(net 22)
+	)
 	(segment
-		(start 130 90)
-		(end 127.38 87.38)
+		(start 127.38 88.88)
+		(end 127.38 84.8)
 		(width 0.5)
-		(layer "F.Cu")
+		(layer "B.Cu")
 		(net 22)
 	)
 	(segment
-		(start 145.36 92.42)
-		(end 139.02 92.42)
+		(start 128.5 90)
+		(end 127.38 88.88)
 		(width 0.5)
-		(layer "F.Cu")
+		(layer "B.Cu")
 		(net 22)
 	)
