File: pcb/bot/esp32_blinds_controller.kicad_pcb (KiCad board)
At the start: 2 copper layers, 100 x 83.2 mm, 42 parts, among them J1 Conn_01x05_Pin, K1 LEG-24, K2 LEG-24, K3 LEG-24, K4 LEG-24, U1 MCP23008-xP, U2 ULN2003A, U3 R-78E3.3-1.0, U4 EL817, U5 EL817, U6 EL817, U7 EL817

Commit message: update
Parts:
- added J2: Conn_01x05_Pin, Connector_JST:JST_EH_B2B-EH-A_1x02_P2.50mm_Vertical, F.Cu at (90.6, 77.0)
- added JP1: Jumper_2_Bridged, Jumper:SolderJumper-2_P1.3mm_Bridged2Bar_Pad1.0x1.5mm, F.Cu at (89.2, 82.0)
- J1: footprint Connector_PinHeader_2.54mm:PinHeader_1x05_P2.54mm_Vertical -> Connector_JST:JST_EH_B6B-EH-A_1x06_P2.50mm_Vertical
- moved J1 47.9 mm to (83.1, 71.1), turned to 0 degrees
- moved K1 4.05 mm to (118.3, 107.3)
- moved K2 4.05 mm to (137.2, 107.3)
- moved K3 4.05 mm to (164.8, 107.3)
- moved K4 4.05 mm to (183.8, 107.3)
Other:
- board text removed: "DOWN"
- board text removed: "LIVE"
- board text removed: "SW"
- board text removed: "UP"
