File: pcb/bot/esp32_blinds_controller.kicad_pcb (KiCad board)
At the start: 2 copper layers, 100 x 83.2 mm, 42 parts, among them J1 Conn_01x05_Pin, K1 LEG-24, K2 LEG-24, K3 LEG-24, K4 LEG-24, U1 MCP23008-xP, U2 ULN2003A, U3 R-78E3.3-1.0, U4 EL817, U5 EL817, U6 EL817, U7 EL817

Commit message: update
Parts:
- U1: footprint Package_DIP:DIP-18_W7.62mm_LongPads -> Package_SO:SOIC-18W_7.5x11.6mm_P1.27mm
- U2: footprint Package_DIP:DIP-16_W7.62mm_LongPads -> Package_SO:SOIC-16_3.9x9.9mm_P1.27mm
- moved U1 20.9 mm to (145.1, 88.8)
- moved U2 14.4 mm to (121.7, 90.5)
- moved K1 4.37 mm to (118.4, 107.6)
- moved K2 4.37 mm to (137.3, 107.6)
- moved K3 4.37 mm to (164.8, 107.6)
- moved K4 4.37 mm to (183.8, 107.6)
Connections:
- U1 pad 10: /UP2 -> /IN4_L
- U1 pad 17: /IN4_L -> /UP2
Routing:
- net /IN4_L: track 43.3 -> 6.95 mm
- net /IN3_L: track 40.5 -> 6.95 mm
- net /IN2_L: track 37.4 -> 6.89 mm
- net /IN1_L: track 34.5 -> 6.88 mm
- net /A0: track 26.3 -> 0.00 mm
- net /A2: track 29.6 -> 5.79 mm
- net /A1: track 27.8 -> 4.33 mm
- net /DN1: track 40.3 -> 30.6 mm
- net /UP2: track 23.5 -> 32.0 mm, vias 1 -> 0
- net +3V3: track 189.1 -> 183.9 mm
- net /UP1: track 33.2 -> 28.0 mm
- net /nUP2: track 72.3 -> 77.4 mm, vias 0 -> 1
- net /DN2: track 29.4 -> 24.9 mm, vias 1 -> 0
- net /L2-SW: track 21.8 -> 17.2 mm
- net /L2-UP: track 21.6 -> 17.1 mm
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- removed copper zone on B.Cu, net GND
- removed copper zone on F.Cu, net GND
Other:
- board text removed: "DOWN"
- board text removed: "LIVE"
- board text removed: "SW"
- board text removed: "UP"

Commit message: UPDATE
Parts:
- added R12: 2.2k, Resistor_SMD:R_0805_2012Metric, F.Cu at (186.6, 69.2)
- added R13: 2.2k, Resistor_SMD:R_0805_2012Metric, F.Cu at (176.8, 69.3)
- added R14: 2.2k, Resistor_SMD:R_0805_2012Metric, F.Cu at (181.5, 69.3)
- added R15: 2.2k, Resistor_SMD:R_0805_2012Metric, F.Cu at (190.7, 69.2)
- C1, C2, C3: footprint Capacitor_THT:C_Disc_D5.0mm_W2.5mm_P5.00mm -> Capacitor_SMD:C_0805_2012Metric
- C4, C5: footprint Capacitor_THT:CP_Radial_D8.0mm_P3.50mm -> Capacitor_SMD:CP_Elec_6.3x7.7
- D10, D5, D6, D7, D8, D9: footprint Diode_THT:D_DO-15_P3.81mm_Vertical_KathodeUp -> Diode_SMD:D_SOD-123
- R1, R2, R3, R4, R5, R6, R7: footprint Resistor_THT:R_Axial_DIN0207_L6.3mm_D2.5mm_P2.54mm_Vertical -> Resistor_SMD:R_0805_2012Metric
- R10, R11, R8, R9: value 4.7K -> 2.2k; footprint Resistor_THT:R_Axial_DIN0207_L6.3mm_D2.5mm_P2.54mm_Vertical -> Resistor_SMD:R_0805_2012Metric
- U4, U5, U6, U7: footprint Package_DIP:DIP-4_W7.62mm -> Package_DIP:SMDIP-4_W9.53mm
- moved A2 19.5 mm to (158.6, 83.8), turned to 0 degrees
- moved C2 19.1 mm to (113.0, 71.7), turned to 90 degrees
- moved C3 16.1 mm to (152.4, 92.9), turned to 90 degrees
- moved D8 11.9 mm to (155.4, 70.7)
- moved D6 11.4 mm to (150.5, 70.6), turned to 0 degrees
- moved A1 10.6 mm to (164.8, 83.8), turned to 0 degrees
- moved D10 9.44 mm to (145.5, 70.7)
- moved D5 7.72 mm to (150.4, 68.2), turned to 180 degrees
- moved D9 7.60 mm to (145.5, 68.2)
- moved D7 7.32 mm to (155.4, 68.2)
- moved R1 6.30 mm to (156.2, 73.0)
- moved R8 6.16 mm to (188.7, 69.2)
- moved R2 5.38 mm to (149.8, 72.8), turned to 180 degrees
- moved C5 4.95 mm to (110.0, 78.0), turned to -90 degrees
- moved D4 4.85 mm to (149.0, 105.0)
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Connections:
- R8 pad 2: /IN2_H -> /IN3_H
- R9 pad 2: /IN3_H -> /IN2_H
- U4 pad 2: GND -> Net-(R13-Pad1)
- U5 pad 1: Net-(R8-Pad1) -> Net-(R9-Pad1)
- U5 pad 2: GND -> Net-(R14-Pad1)
- U6 pad 1: Net-(R9-Pad1) -> Net-(R8-Pad1)
- U6 pad 2: GND -> Net-(R12-Pad1)
- U7 pad 2: GND -> Net-(R15-Pad1)
Routing:
- net /IN4_L: track 6.95 -> 66.7 mm, vias 0 -> 2
- net /IN3_L: track 6.95 -> 51.9 mm, vias 0 -> 2
- net /IN2_L: track 6.89 -> 47.4 mm, vias 0 -> 2
- net /IN1_L: track 6.88 -> 43.9 mm, vias 0 -> 2
- net /A0: track 0.00 -> 31.1 mm, vias 0 -> 1
- net GND: track 0.00 -> 23.9 mm, vias 22 -> 28
- net /A1: track 4.33 -> 23.2 mm, vias 0 -> 1
- net /SDA: track 51.6 -> 39.9 mm
- net /nUP1: track 33.7 -> 43.1 mm
- net /A2: track 5.79 -> 14.6 mm, vias 0 -> 1
- net Net-(R15-Pad1): track 0.00 -> 8.44 mm
- net +3V3: track 183.9 -> 192.0 mm, vias 4 -> 12
- net Net-(R12-Pad1): track 0.00 -> 7.76 mm
- net VBUS: track 260.7 -> 268.4 mm
- net Net-(R14-Pad1): track 0.00 -> 7.32 mm
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- added copper zone on B.Cu, net GND
- added copper zone on F.Cu, net GND
