File: pcb/bot/esp32_blinds_controller.kicad_pcb (KiCad board)
At the start: 2 copper layers, 100 x 83.2 mm, 46 parts, among them J1 Conn_01x05_Pin, K1 LEG-24, K2 LEG-24, K3 LEG-24, K4 LEG-24, U1 MCP23008-xP, U2 ULN2003A, U3 R-78E3.3-1.0, U4 EL817, U5 EL817, U6 EL817, U7 EL817

Commit message: update
Parts:
- J1: footprint Connector_PinHeader_2.54mm:PinHeader_1x05_P2.54mm_Vertical -> Connector_JST:JST_EH_B6B-EH-A_1x06_P2.50mm_Vertical
- moved C1 7.47 mm to (122.7, 78.6), turned to -90 degrees
- moved D10 4.40 mm to (149.9, 70.7)
- moved D5 4.40 mm to (154.8, 68.2)
- moved D6 4.40 mm to (154.9, 70.6)
- moved D7 4.40 mm to (159.8, 68.2)
- moved D8 4.40 mm to (159.8, 70.7)
- moved D9 4.40 mm to (149.9, 68.2)
- moved R1 4.40 mm to (160.6, 73.0)
- moved R3 4.40 mm to (150.6, 72.9)
- moved R2 4.40 mm to (154.2, 72.8)
- moved J1 0.13 mm to (130.8, 69.4), turned to 0 degrees
Routing:
- net VBUS: track 268.4 -> 282.2 mm, vias 1 -> 2
- net /INT: track 46.1 -> 54.9 mm
- net +3V3: track 192.0 -> 199.2 mm
- net /SCL: track 49.3 -> 55.8 mm
- net /SDA: track 39.9 -> 45.9 mm
- net GND: track 23.9 -> 22.2 mm, vias 28 -> 26
