File: pcb/top/esp32_blinds_controller.kicad_pcb (KiCad board)
At the start: 2 copper layers, 100 x 68.2 mm, 29 parts, among them J1 Conn_01x05_Pin, J2 Conn_01x05_Pin, K1 LEG-24, K2 LEG-24, K3 LEG-24, K4 LEG-24, U1 MCP23008-xP, U2 ULN2003A, U3 LTV-847

Commit message: update
Connections:
- U1 pad 10: /UP2 -> /IN4_L
- U1 pad 17: /IN4_L -> /UP2
Routing:
- net /UP2: track 18.2 -> 39.0 mm
- net /IN4_L: track 48.8 -> 67.3 mm
- net GND: vias 43 -> 42
Changed lines of the file:
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@@
 			(layers "*.Cu" "*.Mask")
 			(remove_unused_layers no)
-			(net 22 "/UP2")
+			(net 35 "/IN4_L")
 			(pinfunction "GP0")
 			(pintype "bidirectional")
@@
 			(layers "*.Cu" "*.Mask")
 			(remove_unused_layers no)
-			(net 35 "/IN4_L")
+			(net 22 "/UP2")
 			(pinfunction "GP7")
 			(pintype "bidirectional")
@@
 	)
 	(via
-		(at 143.4 92.7)
-		(size 0.6)
-		(drill 0.3)
-		(layers "F.Cu" "B.Cu")
-		(free yes)
-		(net 2)
-	)
-	(via
 		(at 143.9 75.9)
 		(size 0.6)
@@
 	)
 	(segment
-		(start 139.575 88.375)
-		(end 129.8 88.375)
+		(start 128.905 83.285)
+		(end 128.905 87.48)
 		(width 0.2)
 		(layer "B.Cu")
@@
 	)
 	(segment
-		(start 140.52 90.905)
-		(end 140.52 89.32)
+		(start 139.2 93)
+		(end 157.2 93)
+		(width 0.2)
+		(layer "B.Cu")
+		(net 22)
+	)
+	(segment
+		(start 157.2 93)
+		(end 158.3 91.9)
 		(width 0.2)
 		(layer "B.Cu")
@@
 	(segment
 		(start 129.8 88.375)
-		(end 128.905 87.48)
+		(end 137.375 88.375)
+		(width 0.2)
+		(layer "B.Cu")
+		(net 22)
+	)
+	(segment
+		(start 138.6 92.4)
+		(end 139.2 93)
 		(width 0.2)
 		(layer "B.Cu")
@@
 	(segment
 		(start 128.905 87.48)
-		(end 128.905 83.285)
+		(end 129.8 88.375)
+		(width 0.2)
+		(layer "B.Cu")
+		(net 22)
+	)
+	(segment
+		(start 138.6 89.6)
+		(end 138.6 92.4)
 		(width 0.2)
 		(layer "B.Cu")
@@
 	)
 	(segment
-		(start 140.52 89.32)
-		(end 139.575 88.375)
+		(start 137.375 88.375)
+		(end 138.6 89.6)
+		(width 0.2)
+		(layer "B.Cu")
+		(net 22)
+	)
+	(segment
+		(start 158.3 91.9)
+		(end 158.3 90.905)
 		(width 0.2)
 		(layer "B.Cu")
@@
 	)
 	(segment
-		(start 158.2 86.6)
-		(end 158.3 86.7)
-		(width 0.2)
-		(layer "F.Cu")
-		(net 35)
-	)
-	(segment
 		(start 171.6 80.395)
 		(end 171.6 86.6)
@@
 		(net 35)
 	)
-	(segment
-		(start 158.3 86.7)
-		(end 158.3 90.905)
-		(width 0.2)
-		(layer "F.Cu")
-		(net 35)
-	)
 	(via
 		(at 171.6 86.6)
@@
 	)
 	(via
-		(at 158.2 86.6)
+		(at 140.6 86)
 		(size 0.6)
 		(drill 0.3)
@@
 	)
 	(segment
+		(start 171.6 86.6)
+		(end 142.936764 86.6)
+		(width 0.2)
+		(layer "B.Cu")
+		(net 35)
+	)
+	(segment
 		(start 192.14 86.6)
 		(end 171.6 86.6)
@@
 	)
 	(segment
-		(start 171.6 86.6)
-		(end 158.2 86.6)
+		(start 140.52 90.905)
+		(end 140.6 90.825)
+		(width 0.2)
+		(layer "B.Cu")
+		(net 35)
+	)
+	(segment
+		(start 142.336764 86)
+		(end 140.6 86)
+		(width 0.2)
+		(layer "B.Cu")
+		(net 35)
+	)
+	(segment
+		(start 140.6 90.825)
+		(end 140.6 86)
+		(width 0.2)
+		(layer "B.Cu")
+		(net 35)
+	)
+	(segment
+		(start 142.936764 86.6)
+		(end 142.336764 86)
 		(width 0.2)
 		(layer "B.Cu")
