File: pcb/top/esp32_blinds_controller.kicad_pcb (KiCad board)
At the start: 2 copper layers, 100 x 68.2 mm, 29 parts, among them J1 Conn_01x05_Pin, J2 Conn_01x05_Pin, K1 LEG-24, K2 LEG-24, K3 LEG-24, K4 LEG-24, U1 MCP23008-xP, U2 ULN2003A, U3 LTV-847

Commit message: update
Parts:
- removed U3: LTV-847, Package_DIP:DIP-16_W7.62mm
- added C1: 100nF, Capacitor_SMD:C_0805_2012Metric, F.Cu at (219.8, 97.2)
- added R1: 4.7K, Resistor_SMD:R_0805_2012Metric, F.Cu at (219.8, 76.5)
- added R12: 2.2k, Resistor_SMD:R_0805_2012Metric, F.Cu at (219.8, 85.4)
- added R13: 2.2k, Resistor_SMD:R_0805_2012Metric, F.Cu at (219.8, 88.3)
- added R14: 2.2k, Resistor_SMD:R_0805_2012Metric, F.Cu at (219.8, 91.3)
- added R15: 2.2k, Resistor_SMD:R_0805_2012Metric, F.Cu at (219.8, 94.2)
- added R2: 4.7K, Resistor_SMD:R_0805_2012Metric, F.Cu at (219.8, 79.5)
- added R3: 4.7K, Resistor_SMD:R_0805_2012Metric, F.Cu at (219.8, 82.4)
- added U4: EL817, Package_DIP:SMDIP-4_W9.53mm, F.Cu at (211.0, 78.4)
- added U5: EL817, Package_DIP:SMDIP-4_W9.53mm, F.Cu at (211.0, 85.0)
- added U6: EL817, Package_DIP:SMDIP-4_W9.53mm, F.Cu at (211.0, 91.6)
- added U7: EL817, Package_DIP:SMDIP-4_W9.53mm, F.Cu at (211.0, 98.3)
- C2, C3: footprint Capacitor_THT:C_Disc_D5.0mm_W2.5mm_P5.00mm -> Capacitor_SMD:C_0805_2012Metric
- C4, C5: footprint Capacitor_THT:CP_Radial_D8.0mm_P3.50mm -> Capacitor_SMD:CP_Elec_6.3x7.7
- R10, R11, R8, R9: value 4.7K -> 2.2k; footprint Resistor_THT:R_Axial_DIN0207_L6.3mm_D2.5mm_P2.54mm_Vertical -> Resistor_SMD:R_0805_2012Metric
- R4, R5, R6, R7: footprint Resistor_THT:R_Axial_DIN0207_L6.3mm_D2.5mm_P2.54mm_Vertical -> Resistor_SMD:R_0805_2012Metric
- U1: footprint Package_DIP:DIP-18_W7.62mm_LongPads -> Package_SO:SOIC-18W_7.5x11.6mm_P1.27mm
- U2: footprint Package_DIP:DIP-16_W7.62mm_LongPads -> Package_SO:SOIC-16_3.9x9.9mm_P1.27mm
- moved C4 27.6 mm to (125.0, 87.0), turned to 180 degrees
- moved C3 23.1 mm to (169.7, 86.0)
- moved C2 7.92 mm to (107.8, 87.1)
- moved C5 5.78 mm to (115.3, 87.0)
- moved U1 4.48 mm to (158.5, 87.1)
- moved U2 4.29 mm to (137.1, 88.6)
Connections:
- R8 pad 2: /IN2_H -> /IN3_H
- R9 pad 2: /IN3_H -> /IN2_H
- U2 pad 4: /UP2 -> unconnected-(U2-I4-Pad4)
- U2 pad 5: /DN2 -> unconnected-(U2-I5-Pad5)
- U2 pad 6: /UP1 -> unconnected-(U2-I6-Pad6)
- U2 pad 7: /DN1 -> unconnected-(U2-I7-Pad7)
Routing:
- net /IN4_L: track 67.3 -> 0.00 mm, vias 3 -> 0
- net +3V3: track 85.7 -> 36.8 mm, vias 1 -> 0
- net /IN3_L: track 45.5 -> 0.06 mm, vias 3 -> 0
- net /IN2_L: track 42.4 -> 0.03 mm, vias 3 -> 0
- net /IN1_L: track 39.2 -> 0.00 mm, vias 3 -> 0
- net /UP2: track 39.0 -> 0.00 mm
- net /DN1: track 33.5 -> 4.17 mm, vias 1 -> 0
- net /UP1: track 27.9 -> 0.00 mm, vias 1 -> 0
- net /DN2: track 23.1 -> 0.00 mm, vias 1 -> 0
- net /nUP1: track 32.4 -> 22.8 mm
- net /nUP2: track 74.4 -> 65.6 mm
- net /nDOWN2: track 54.4 -> 46.1 mm
- net /nDOWN1: track 12.9 -> 19.8 mm
- net VBUS: track 237.7 -> 235.1 mm
- net GND: vias 42 -> 12
- removed copper zone on B.Cu, net GND
- removed copper zone on F.Cu, net GND

Commit message: update
Parts:
- moved C1 69.3 mm to (154.4, 74.1), turned to 90 degrees
- moved R3 61.4 mm to (158.7, 75.9), turned to -90 degrees
- moved R2 59.2 mm to (160.7, 75.9), turned to -90 degrees
- moved R1 57.0 mm to (162.8, 75.9), turned to -90 degrees
- moved R13 45.0 mm to (176.5, 75.9), turned to 90 degrees
- moved R14 41.1 mm to (181.6, 75.9), turned to 90 degrees
- moved R12 34.9 mm to (186.2, 75.9), turned to 90 degrees
- moved U4 34.6 mm to (177.7, 87.6), turned to -90 degrees
- moved R15 34.5 mm to (190.5, 75.9), turned to 90 degrees
- moved U5 27.6 mm to (183.5, 87.6), turned to -90 degrees
- moved U6 22.1 mm to (189.3, 87.6), turned to -90 degrees
- moved U7 19.1 mm to (195.1, 87.6), turned to -90 degrees
- moved R6 16.2 mm to (171.6, 91.2), turned to 90 degrees
- moved R4 14.3 mm to (173.6, 91.2), turned to 90 degrees
- moved R7 14.0 mm to (167.4, 91.2), turned to 90 degrees
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Connections:
- U2 pad 4: unconnected-(U2-I4-Pad4) -> /UP2
- U2 pad 5: unconnected-(U2-I5-Pad5) -> /DN2
- U2 pad 6: unconnected-(U2-I6-Pad6) -> /UP1
- U2 pad 7: unconnected-(U2-I7-Pad7) -> /DN1
Routing:
- net +3V3: track 36.8 -> 97.2 mm, vias 0 -> 3
- net /IN4_L: track 0.00 -> 58.9 mm, vias 0 -> 3
- net /IN3_L: track 0.06 -> 43.7 mm, vias 0 -> 3
- net /IN2_L: track 0.03 -> 37.0 mm, vias 0 -> 3
- net /UP2: track 0.00 -> 32.3 mm, vias 0 -> 2
- net /IN1_L: track 0.00 -> 30.4 mm, vias 0 -> 3
- net /DN1: track 4.17 -> 28.9 mm, vias 0 -> 2
- net /UP1: track 0.00 -> 24.8 mm, vias 0 -> 2
- net GND: track 5.00 -> 27.9 mm, vias 12 -> 24
- net /DN2: track 0.00 -> 22.9 mm, vias 0 -> 2
- net /INT: track 34.8 -> 53.8 mm, vias 0 -> 2
- net /A2: track 21.7 -> 29.6 mm
- net Net-(R15-Pad1): track 0.00 -> 7.50 mm
- net /A0: track 25.3 -> 32.3 mm
- net /A1: track 24.0 -> 30.8 mm
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- added copper zone on B.Cu, net GND
- added copper zone on F.Cu, net GND
