File: pcb/top/esp32_blinds_controller.kicad_pcb (KiCad board)
At the start: 2 copper layers, 100 x 60 mm, 31 parts, among them J1 Conn_01x05_Pin, K1 LEG-24, K2 LEG-24, K3 LEG-24, K4 LEG-24, U1 MCP23008-xP, U2 ULN2003A

Commit message: update
Parts:
- removed C1: 100nF, Capacitor_THT:C_Disc_D5.0mm_W2.5mm_P5.00mm
- removed R1, R2, R3: 4.7K, Resistor_THT:R_Axial_DIN0207_L6.3mm_D2.5mm_P2.54mm_Vertical
- added U3: LTV-847, Package_DIP:DIP-16_W7.62mm, F.Cu at (192.1, 83.3)
- A0, A1, A2: moved to B.Cu
- moved R11 125.0 mm to (192.0, 77.9), turned to 90 degrees
- moved R9 121.5 mm to (188.7, 77.9), turned to 90 degrees
- moved R8 116.5 mm to (183.6, 77.9), turned to 90 degrees
- moved R10 111.4 mm to (178.6, 77.9), turned to 90 degrees
- moved R4 107.6 mm to (168.6, 77.9), turned to -90 degrees
- moved R7 104.8 mm to (171.6, 77.9), turned to -90 degrees
- moved R5 104.6 mm to (165.5, 77.9), turned to -90 degrees
- moved R6 101.9 mm to (162.4, 77.9), turned to -90 degrees
- moved C4 78.5 mm to (149.3, 74.0)
- moved A2 75.8 mm to (138.7, 76.2), turned to 90 degrees
- moved J1 75.3 mm to (127.1, 77.2), turned to -90 degrees
- moved A1 71.7 mm to (135.5, 76.2), turned to 90 degrees
- moved C3 67.5 mm to (147.4, 80.1)
- moved A0 67.3 mm to (131.9, 76.3), turned to 90 degrees
- moved D1 4.90 mm to (127.6, 99.5)
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Routing:
- net +3V3: track 24.8 -> 84.1 mm, vias 0 -> 1
- net /IN4_L: track 0.00 -> 49.5 mm, vias 0 -> 3
- net /IN3_L: track 0.00 -> 46.4 mm, vias 0 -> 3
- net /IN2_L: track 0.00 -> 43.2 mm, vias 0 -> 3
- net /IN1_L: track 0.00 -> 40.3 mm, vias 0 -> 3
- net /SCL: track 21.1 -> 56.5 mm, vias 0 -> 2
- net /SDA: track 24.6 -> 52.3 mm, vias 0 -> 2
- net /A0: track 0.00 -> 25.3 mm, vias 0 -> 1
- net /A1: track 0.00 -> 23.4 mm, vias 0 -> 1
- net /A2: track 0.00 -> 21.3 mm, vias 0 -> 1
- net /INT: track 14.7 -> 32.7 mm
- net /IN4_H: track 0.00 -> 7.44 mm
- net /IN3_H: track 0.00 -> 6.81 mm
- net /IN2_H: track 0.00 -> 6.78 mm
- net /IN1_H: track 0.00 -> 6.68 mm
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- added copper zone on B.Cu, net GND
- added copper zone on F.Cu, net GND
Other:
- board size 100 x 60 mm -> 100 x 68.2 mm
- board text added: "REV ${Revision} TOP"
- board text removed: "1"
- board text removed: "REV ${Revision}"

Commit message: update
Parts:
- added J2: Conn_01x05_Pin, Connector_JST:JST_EH_B6B-EH-A_1x06_P2.50mm_Vertical, F.Cu at (127.2, 76.0)
- J1: footprint Connector_PinHeader_2.54mm:PinHeader_1x05_P2.54mm_Vertical -> Connector_JST:JST_EH_B6B-EH-A_1x06_P2.50mm_Vertical; moved to B.Cu
- moved J1 1.80 mm to (127.2, 79.0), turned to 180 degrees
Routing:
- net +3V3: track 84.1 -> 86.5 mm

Commit message: update
Parts:
- moved U2 1.09 mm to (136.5, 84.4)
- moved J1 1.00 mm to (127.2, 80.0)
- moved U1 0.82 mm to (160.8, 83.3)
- moved J2 0.80 mm to (127.2, 76.8)
Routing:
- net VBUS: track 230.4 -> 237.7 mm
- net /INT: track 32.7 -> 34.8 mm
- net /SDA: track 52.3 -> 54.4 mm
- net /SCL: track 56.5 -> 58.5 mm
- net /IN1_L: track 40.3 -> 39.2 mm
- net /DN1: track 32.5 -> 33.5 mm
- net /IN3_L: track 46.4 -> 45.5 mm
- net /UP2: track 17.3 -> 18.2 mm
- net +3V3: track 86.5 -> 85.7 mm
- net /IN2_L: track 43.2 -> 42.4 mm
- net /IN4_L: track 49.5 -> 48.8 mm
- net /A1: track 23.4 -> 24.0 mm
- net GND: vias 45 -> 43

Commit message: update
Connections:
- U1 pad 10: /UP2 -> /IN4_L
- U1 pad 17: /IN4_L -> /UP2
Routing:
- net /UP2: track 18.2 -> 36.3 mm, vias 0 -> 1
- net /IN4_L: track 48.8 -> 66.6 mm, vias 3 -> 2
- net GND: vias 43 -> 39
Changed lines of the file:
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@@
 		(allow_soldermask_bridges_in_footprints no)
 		(pcbplotparams
-			(layerselection 0x00010fc_ffffffff)
-			(plot_on_all_layers_selection 0x0001000_00000000)
+			(layerselection 0x00011fc_ffffffff)
+			(plot_on_all_layers_selection 0x0001020_00000000)
 			(disableapertmacros no)
 			(usegerberextensions no)
@@
 			(dashed_line_gap_ratio 3.000000)
 			(svgprecision 4)
-			(plotframeref no)
+			(plotframeref yes)
 			(viasonmask no)
 			(mode 1)
@@
 			(sketchpadsonfab no)
 			(subtractmaskfromsilk no)
-			(outputformat 1)
+			(outputformat 4)
 			(mirror no)
 			(drillshape 0)
@@
 			(layers "*.Cu" "*.Mask")
 			(remove_unused_layers no)
-			(net 22 "/UP2")
+			(net 35 "/IN4_L")
 			(pinfunction "GP0")
 			(pintype "bidirectional")
@@
 			(layers "*.Cu" "*.Mask")
 			(remove_unused_layers no)
-			(net 35 "/IN4_L")
+			(net 22 "/UP2")
 			(pinfunction "GP7")
 			(pintype "bidirectional")
@@
 		)
 	)
+	(dimension
+		(type aligned)
+		(layer "Dwgs.User")
+		(pts
+			(xy 101.175 131.37) (xy 201.175 131.37)
+		)
+		(height 4.229999)
+		(gr_text "100.0000 mm"
+			(at 151.175 134.449999 0)
+			(layer "Dwgs.User")
+			(effects
+				(font
+					(size 1 1)
+					(thickness 0.15)
+				)
+			)
+		)
+		(format
+			(prefix "")
+			(suffix "")
+			(units 3)
+			(units_format 1)
+			(precision 4)
+		)
+		(style
+			(thickness 0.1)
+			(arrow_length 1.27)
+			(text_position_mode 0)
+			(extension_height 0.58642)
+			(extension_offset 0.5) keep_text_aligned)
+	)
+	(dimension
+		(type aligned)
+		(layer "Dwgs.User")
+		(pts
+			(xy 201.175 63.12) (xy 201.175 131.37)
+		)
+		(height -4.475)
+		(gr_text "68.2500 mm"
+			(at 204.5 97.245 90)
+			(layer "Dwgs.User")
+			(effects
+				(font
+					(size 1 1)
+					(thickness 0.15)
+				)
+			)
+		)
+		(format
+			(prefix "")
+			(suffix "")
+			(units 3)
+			(units_format 1)
+			(precision 4)
+		)
+		(style
+			(thickness 0.1)
+			(arrow_length 1.27)
+			(text_position_mode 0)
+			(extension_height 0.58642)
+			(extension_offset 0.5) keep_text_aligned)
+	)
 	(segment
 		(start 124.4 114.55)
@@
 	)
 	(via
-		(at 151 85)
-		(size 0.6)
-		(drill 0.3)
-		(layers "F.Cu" "B.Cu")
-		(free yes)
-		(net 2)
-	)
-	(via
 		(at 102.1 64)
 		(size 0.6)
@@
 	)
 	(via
-		(at 145.5 85)
-		(size 0.6)
-		(drill 0.3)
-		(layers "F.Cu" "B.Cu")
-		(free yes)
-		(net 2)
-	)
-	(via
 		(at 174.1 81.5)
 		(size 0.6)
@@
 	)
 	(via
-		(at 156 85)
-		(size 0.6)
-		(drill 0.3)
-		(layers "F.Cu" "B.Cu")
-		(free yes)
-		(net 2)
-	)
-	(via
 		(at 180.1 81.2)
 		(size 0.6)
@@
 	)
 	(via
-		(at 158.5 85)
-		(size 0.6)
-		(drill 0.3)
-		(layers "F.Cu" "B.Cu")
-		(free yes)
-		(net 2)
-	)
-	(via
 		(at 164 89.5)
 		(size 0.6)
@@
 	)
 	(segment
-		(start 139.575 88.375)
-		(end 129.8 88.375)
+		(start 158.3 86.6)
+		(end 158.3 90.905)
+		(width 0.2)
+		(layer "F.Cu")
+		(net 22)
+	)
+	(segment
+		(start 157.4 85.7)
+		(end 158.3 86.6)
+		(width 0.2)
+		(layer "F.Cu")
+		(net 22)
+	)
+	(via
+		(at 157.4 85.7)
+		(size 0.6)
+		(drill 0.3)
+		(layers "F.Cu" "B.Cu")
+		(net 22)
+	)
+	(segment
+		(start 157.4 85.7)
+		(end 141.25 85.7)
 		(width 0.2)
 		(layer "B.Cu")
@@
 	)
 	(segment
-		(start 140.52 90.905)
-		(end 140.52 89.32)
+		(start 128.905 85.855)
+		(end 128.905 84.375)
 		(width 0.2)
 		(layer "B.Cu")
@@
 	)
 	(segment
-		(start 129.8 88.375)
-		(end 128.905 87.48)
+		(start 129.75 86.7)
+		(end 128.905 85.855)
 		(width 0.2)
 		(layer "B.Cu")
@@
 	)
 	(segment
-		(start 128.905 87.48)
-		(end 128.905 83.285)
+		(start 140.25 86.7)
+		(end 129.75 86.7)
 		(width 0.2)
 		(layer "B.Cu")
@@
 	)
 	(segment
-		(start 140.52 89.32)
-		(end 139.575 88.375)
+		(start 141.25 85.7)
+		(end 140.25 86.7)
 		(width 0.2)
 		(layer "B.Cu")
@@
 	)
 	(segment
-		(start 158.2 86.6)
-		(end 158.3 86.7)
-		(width 0.2)
-		(layer "F.Cu")
-		(net 35)
-	)
-	(segment
 		(start 171.6 80.395)
 		(end 171.6 86.6)
@@
 		(net 35)
 	)
-	(segment
-		(start 158.3 86.7)
-		(end 158.3 90.905)
-		(width 0.2)
-		(layer "F.Cu")
-		(net 35)
-	)
 	(via
 		(at 171.6 86.6)
@@
 	)
 	(via
-		(at 158.2 86.6)
+		(at 192.14 86.6)
 		(size 0.6)
 		(drill 0.3)
@@
 		(net 35)
 	)
-	(via
-		(at 192.14 86.6)
-		(size 0.6)
-		(drill 0.3)
-		(layers "F.Cu" "B.Cu")
+	(segment
+		(start 141.55 86.15)
+		(end 156.4 86.15)
+		(width 0.2)
+		(layer "B.Cu")
+		(net 35)
+	)
+	(segment
+		(start 156.95 86.7)
+		(end 165.151471 86.7)
+		(width 0.2)
+		(layer "B.Cu")
+		(net 35)
+	)
+	(segment
+		(start 140.52 87.18)
+		(end 141.55 86.15)
+		(width 0.2)
+		(layer "B.Cu")
+		(net 35)
+	)
+	(segment
+		(start 156.4 86.15)
+		(end 156.95 86.7)
+		(width 0.2)
+		(layer "B.Cu")
 		(net 35)
 	)
@@
 	)
 	(segment
-		(start 171.6 86.6)
-		(end 158.2 86.6)
+		(start 140.52 90.905)
+		(end 140.52 87.18)
+		(width 0.2)
+		(layer "B.Cu")
+		(net 35)
+	)
+	(segment
+		(start 165.251471 86.6)
+		(end 171.6 86.6)
+		(width 0.2)
+		(layer "B.Cu")
+		(net 35)
+	)
+	(segment
+		(start 165.151471 86.7)
+		(end 165.251471 86.6)
 		(width 0.2)
 		(layer "B.Cu")

Commit message: update
Parts:
- removed U3: LTV-847, Package_DIP:DIP-16_W7.62mm
- added C1: 100nF, Capacitor_SMD:C_0805_2012Metric, F.Cu at (154.4, 74.1)
- added R1: 4.7K, Resistor_SMD:R_0805_2012Metric, F.Cu at (162.8, 75.9)
- added R12: 2.2k, Resistor_SMD:R_0805_2012Metric, F.Cu at (186.2, 75.9)
- added R13: 2.2k, Resistor_SMD:R_0805_2012Metric, F.Cu at (176.5, 75.9)
- added R14: 2.2k, Resistor_SMD:R_0805_2012Metric, F.Cu at (181.6, 75.9)
- added R15: 2.2k, Resistor_SMD:R_0805_2012Metric, F.Cu at (190.5, 75.9)
- added R2: 4.7K, Resistor_SMD:R_0805_2012Metric, F.Cu at (160.7, 75.9)
- added R3: 4.7K, Resistor_SMD:R_0805_2012Metric, F.Cu at (158.7, 75.9)
- added U4: EL817, Package_DIP:SMDIP-4_W9.53mm, F.Cu at (177.7, 87.6)
- added U5: EL817, Package_DIP:SMDIP-4_W9.53mm, F.Cu at (183.5, 87.6)
- added U6: EL817, Package_DIP:SMDIP-4_W9.53mm, F.Cu at (189.3, 87.6)
- added U7: EL817, Package_DIP:SMDIP-4_W9.53mm, F.Cu at (195.1, 87.6)
- C2, C3: footprint Capacitor_THT:C_Disc_D5.0mm_W2.5mm_P5.00mm -> Capacitor_SMD:C_0805_2012Metric
- C4, C5: footprint Capacitor_THT:CP_Radial_D8.0mm_P3.50mm -> Capacitor_SMD:CP_Elec_6.3x7.7
- R10, R11, R8, R9: value 4.7K -> 2.2k; footprint Resistor_THT:R_Axial_DIN0207_L6.3mm_D2.5mm_P2.54mm_Vertical -> Resistor_SMD:R_0805_2012Metric
- R4, R5, R6, R7: footprint Resistor_THT:R_Axial_DIN0207_L6.3mm_D2.5mm_P2.54mm_Vertical -> Resistor_SMD:R_0805_2012Metric
- U1: footprint Package_DIP:DIP-18_W7.62mm_LongPads -> Package_SO:SOIC-18W_7.5x11.6mm_P1.27mm
- U2: footprint Package_DIP:DIP-16_W7.62mm_LongPads -> Package_SO:SOIC-16_3.9x9.9mm_P1.27mm
- moved C4 27.6 mm to (125.0, 87.0), turned to 180 degrees
- moved C3 21.0 mm to (165.2, 91.2), turned to 90 degrees
- moved R6 16.2 mm to (171.6, 91.2), turned to 90 degrees
- moved R4 14.3 mm to (173.6, 91.2), turned to 90 degrees
- moved R7 14.0 mm to (167.4, 91.2), turned to 90 degrees
- moved R5 13.9 mm to (169.5, 91.2), turned to 90 degrees
- moved C2 8.02 mm to (107.8, 87.0)
- moved C5 5.78 mm to (115.3, 87.0)
- moved R9 5.49 mm to (183.6, 75.9)
- moved R8 5.30 mm to (188.5, 75.9)
- moved U1 4.70 mm to (158.1, 87.1)
- moved U2 4.29 mm to (137.1, 88.6)
- moved R11 2.10 mm to (192.5, 75.9)
- moved R10 2.04 mm to (178.6, 75.9)
- moved D1 0.32 mm to (127.6, 99.2)
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Connections:
- R8 pad 2: /IN2_H -> /IN3_H
- R9 pad 2: /IN3_H -> /IN2_H
Routing:
- net GND: track 5.00 -> 27.9 mm, vias 39 -> 24
- net /INT: track 34.8 -> 53.8 mm, vias 0 -> 2
- net +3V3: track 85.7 -> 97.2 mm, vias 1 -> 3
- net /nUP1: track 32.4 -> 21.3 mm, vias 0 -> 1
- net /nDOWN2: track 54.4 -> 44.6 mm, vias 0 -> 1
- net /nUP2: track 74.4 -> 65.6 mm
- net /IN1_L: track 39.2 -> 30.4 mm
- net /A2: track 21.7 -> 29.6 mm
- net /IN4_L: track 66.6 -> 58.9 mm, vias 2 -> 3
- net Net-(R15-Pad1): track 0.00 -> 7.50 mm
- net /A0: track 25.3 -> 32.3 mm
- net /A1: track 24.0 -> 30.8 mm
- net Net-(R12-Pad1): track 0.00 -> 6.79 mm
- net Net-(R14-Pad1): track 0.00 -> 6.28 mm
- net /SDA: track 54.4 -> 60.5 mm, vias 2 -> 3
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